Commit message: Add TCPs

File: rh5_fixed.urdf (robot description, URDF)
Before this commit: robot RH5, 58 links, 57 joints
Links:
- added link LTCP_Link
- added link RTCP_Link
Joints:
- added joint LTCP: type fixed, parent ALWristPitch_Link, child LTCP_Link, origin xyz=0 0 -0.15 rpy=3.1415926 0 1.57, axis 0 0 1.0, limit lower=-1.0 upper=1.0 effort=0 velocity=0
- added joint RTCP: type fixed, parent ARWristPitch_Link, child RTCP_Link, origin xyz=0 0 -0.15 rpy=3.1415926 0 1.57, axis 0 0 1.0, limit lower=-1.0 upper=1.0 effort=0 velocity=0
