Commit message: Start solar panel in pybullet
URDF needs to be fixed

File: rh5_left_arm.urdf (robot description, URDF)
Before this commit: robot RH5, 13 links, 12 joints
Links:
- added link LTCP_Link
Joints:
- added joint LTCP: type fixed, parent ALWristPitch_Link, child LTCP_Link, origin xyz=0 0 -0.15 rpy=3.1415926 0 1.57, axis 0 0 1.0, limit lower=-1.0 upper=1.0 effort=0 velocity=0

File: rh5_right_arm.urdf (robot description, URDF)
Before this commit: robot RH5, 13 links, 12 joints
Links:
- added link RTCP_Link
Joints:
- added joint RTCP: type fixed, parent ARWristPitch_Link, child RTCP_Link, origin xyz=0 0 -0.15 rpy=3.1415926 0 1.57, axis 0 0 1.0, limit lower=-1.0 upper=1.0 effort=0 velocity=0
